Commit message: Documentation added for robot fixed laser and camera issues

File: catbot/robots/catbot.URDF (robot description, URDF)
Before this commit: robot catbot, 7 links, 6 joints
Joints:
- joint ball_and_socket: axis 0 0 -1 -> (none); type continuous -> fixed
- joint base_footprint_joint: origin xyz=0 0 0.11 rpy=0 0 0 -> xyz=0 0 0.13 rpy=0 0 0

Commit message: Version 0.2.0 Fixed issue with node teleop removed transmission tags from nodes removed config file modified gazebo.launch to include the teleop_node

File: catbot/robots/catbot.URDF (robot description, URDF)
Before this commit: robot catbot, 7 links, 6 joints
Joints:
- joint base_footprint_joint: origin xyz=0 0 0.13 rpy=0 0 0 -> xyz=0 0 0.125 rpy=0 0 0

Commit message: Version 0.3.0
fully functional teleop node
fully functional differential robot plugin simulation
yayyy !!!

File: catbot/robots/catbot.URDF (robot description, URDF)
Before this commit: robot catbot, 7 links, 6 joints
Links:
- link left_wheel: mass 0.2 -> 2
- link right_wheel: mass 0.2 -> 2
Joints:
- joint base_footprint_joint: origin xyz=0 0 0.125 rpy=0 0 0 -> xyz=0 0 0.125 rpy=0 0 -1.570796327
- joint left_motor: axis 0 0 -1 -> 0 0 1; limit effort=0.863 velocity=12.57 -> effort=100 velocity=100
- joint right_motor: limit effort=0.863 velocity=12.57 -> effort=100 velocity=100
