Commit message: Added four-wheeled-drive gazebo plugin

File: catbot_description/urdf/catbot.urdf.xacro (robot description, xacro)
@@ -8,5 +8,5 @@
     <property name="base_length" value = "0.60"/>
     <property name="base_height" value = "0.10"/>
-    <property name="base_mass"   value = "1.50"/>
+    <property name="base_mass"   value = "5"/>
     <link name="base_footprint">
         <inertial>
@@ -46,5 +46,5 @@
             iyy = "${base_mass*(base_length*base_length+base_height*base_height)}"
             iyz = "0"
-            izz = "${base_mass*(base_width*base_width+base_length*base_length)}"/>
+            izz = "${base_mass*(base_width*base_width+base_length*base_length)/12}"/>
         </inertial>
         <visual>
@@ -73,3 +73,29 @@
         </plugin>
     </gazebo>
+    <gazebo>
+        <plugin name="differential_drive_controller" filename="libgazebo_ros_four_wheeled_drive.so">
+            <rosDebugLevel> Debug </rosDebugLevel>
+            <publishWheelTF>true</publishWheelTF>
+            <robotNameSpace>/</robotNameSpace>
+            <publishTF>1</publishTF>
+            <publishWheelJointState>true</publishWheelJointState>
+            <alwaysOn>true</alwaysOn>
+            <updateRate>50</updateRate>
+            <frontLeftJoint>front_left_wheel_joint</frontLeftJoint>
+            <frontRightJoint>front_right_wheel_joint</frontRightJoint>
+            <backLeftJoint>back_left_wheel_joint</backLeftJoint>
+            <backRightJoint>back_right_wheel_joint</backRightJoint>
+            <wheelSeparation>0.4</wheelSeparation>
+            <wheelDiameter>0.2</wheelDiameter>
+            <broadcastTF>1</broadcastTF>
+            <wheelTorque>100</wheelTorque>
+            <wheelAcceleration>2.8</wheelAcceleration>
+            <commandTopic>catbot/cmd_vel</commandTopic>
+            <odometryFrame>catbot/odom</odometryFrame>
+            <odometryTopic>catbot/odom</odometryTopic>
+            <robotBaseFrame>base_footprint</robotBaseFrame>
+            <legacyMode>true</legacyMode>
+            <odometrySource>encoder</odometrySource>
+        </plugin>
+    </gazebo>
 </robot>

File: catbot_description/urdf/include/camera.urdf.xacro (robot description, xacro)
@@ -10,5 +10,5 @@
         </visual>
         <inertial>
-            <mass value="0.2" />
+            <mass value="0.02" />
             <inertia
                 ixx="0.0001"

File: catbot_description/urdf/include/laser_scanner.urdf.xacro (robot description, xacro)
@@ -17,5 +17,5 @@
             </collision>
             <inertial>
-                <mass value="0.2" />
+                <mass value="0.02" />
                 <inertia
                     ixx="0.0001"

File: catbot_description/urdf/include/wheel.urdf.xacro (robot description, xacro)
@@ -7,5 +7,5 @@
   <property name="wheel_radius" value="0.10" />
   <property name="wheel_height" value="0.07" />
-  <property name="wheel_mass" value="2.5" /> <!-- in kg-->
+  <property name="wheel_mass" value="0.5" /> <!-- in kg-->
   <property name="base_x_origin_to_wheel_origin" value="0.25" />
   <property name="base_y_origin_to_wheel_origin" value="0.3" />
@@ -38,11 +38,14 @@
     </link>
     <gazebo reference="${fb}_${lr}_wheel">
-      <mu1 value="1.0"/>
-      <mu2 value="1.0"/>
-      <kp  value="10000000.0" />
-      <kd  value="1.0" />
       <fdir1 value="1 0 0"/>
       <material>Gazebo/Black</material>
+      <mu1>1</mu1>
+      <mu2>0</mu2>
+      <kp>1000000.0</kp>
+      <kd>1.0</kd>
+      <minDepth>0.01</minDepth>
+      <maxContacts>1</maxContacts>
       <turnGravityOff>false</turnGravityOff>
+      <dampingFactor>0.01</dampingFactor>
     </gazebo>
     <joint name="${fb}_${lr}_wheel_joint" type="continuous">
@@ -52,9 +55,5 @@
       <axis xyz="0 1 0" rpy="0  0" />
       <limit effort="100" velocity="100"/>
-      <joint_properties damping="15" friction="1"/>
     </joint>
-    <gazebo reference="${fb}_${lr}_wheel_joint">
-        <implicitSpringDamper>true</implicitSpringDamper>
-    </gazebo>
     <!-- Transmission is important to link the joints and the controller -->
     <transmission name="${fb}_${lr}_wheel_joint_trans">
