Commit message: Version 0.5.0

File: catbot_description/urdf/diff_catbot.URDF (robot description, URDF)
Before this commit: robot catbot, 7 links, 6 joints
Links:
- link base_link: geometry collision mesh filename=package://catbot_description/meshes/diff_catbot/base_link.S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; visual mesh filename=package://catbot_description/meshes/diff_catbot/base_link.S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
- link camera: geometry collision mesh filename=package://catbot_description/meshes/diff_catbot/camera.STL; visual mesh filename=package://catbot_description/meshes/diff_catbot/camera.STL
- link caster_wheel: geometry collision mesh filename=package://catbot_description/meshes/diff_catbot/caster_whee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; visual mesh filename=package://catbot_description/meshes/diff_catbot/caster_whee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
- link laser_scanner: geometry collision mesh filename=package://catbot_description/meshes/diff_catbot/laser_scann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; visual mesh filename=package://catbot_description/meshes/diff_catbot/laser_scann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
- link left_wheel: geometry collision mesh filename=package://catbot_description/meshes/diff_catbot/left_wheel.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; visual mesh filename=package://catbot_description/meshes/diff_catbot/left_wheel.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
- link right_wheel: geometry collision mesh filename=package://catbot_description/meshes/diff_catbot/right_wheel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; visual mesh filename=package://catbot_description/meshes/diff_catbot/right_wheel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

File: catbot_description/urdf/fourWD_catbot.urdf.xacro (robot description, xacro)
@@ -1,4 +1,4 @@
 <?xml version="1.0" ?>
-<robot name="catbot" xmlns:xacro="http://ros.org/wiki/xacro">
+<robot name="fourWD_catbot" xmlns:xacro="http://ros.org/wiki/xacro">
     <xacro:include filename="$(find catbot_description)/urdf/include/wheel.urdf.xacro" />
     <xacro:include filename="$(find catbot_description)/urdf/include/laser_scanner.urdf.xacro" />
@@ -14,10 +14,10 @@
             <origin xyz="0 0 0" />
             <inertia
-                ixx="0.0001"
+                ixx="0.0000001"
                 ixy="0.0"
                 ixz="0.0"
-                iyy="0.0001"
+                iyy="0.0000001"
                 iyz="0.0"
-                izz="0.0001" />
+                izz="0.0000001" />
         </inertial>
         <visual>
@@ -41,8 +41,8 @@
             <mass value = "${base_mass}" />
             <inertia
-            ixx = "${base_mass*(base_width*base_width+base_height*base_height)}"
+            ixx = "${base_mass*(base_width*base_width+base_height*base_height)/12}"
             ixy = "0"
             ixz = "0"
-            iyy = "${base_mass*(base_length*base_length+base_height*base_height)}"
+            iyy = "${base_mass*(base_length*base_length+base_height*base_height)/12}"
             iyz = "0"
             izz = "${base_mass*(base_width*base_width+base_length*base_length)/12}"/>
@@ -68,14 +68,14 @@
     <camera_link parent="base_link" x="${(base_length+0.05)/2}" y = "0" z="0" r = "0" p ="0" yaw = "0"/>
     <imu_link parent="base_link" />
-    <gazebo>
+    <!--<gazebo>
         <plugin name="gazebo_ros_control" filename="libgazebo_ros_control.so">
-          <robotNamespace>/catbot</robotNamespace>
+          <robotNamespace>/fourWD_catbot</robotNamespace>
         </plugin>
-    </gazebo>
+    </gazebo> -->
     <gazebo>
         <plugin name="differential_drive_controller" filename="libgazebo_ros_four_wheeled_drive.so">
             <rosDebugLevel> Debug </rosDebugLevel>
             <publishWheelTF>true</publishWheelTF>
-            <robotNameSpace>/</robotNameSpace>
+            <robotNameSpace>/fourWD_catbot</robotNameSpace>
             <publishTF>1</publishTF>
             <publishWheelJointState>true</publishWheelJointState>
@@ -89,6 +89,6 @@
             <wheelDiameter>0.2</wheelDiameter>
             <broadcastTF>1</broadcastTF>
-            <wheelTorque>100</wheelTorque>
-            <wheelAcceleration>2.8</wheelAcceleration>
+            <wheelTorque>30</wheelTorque>
+            <wheelAcceleration>9.8</wheelAcceleration>
             <commandTopic>catbot/cmd_vel</commandTopic>
             <odometryFrame>catbot/odom</odometryFrame>

File: catbot_description/urdf/include/wheel.urdf.xacro (robot description, xacro)
@@ -38,12 +38,11 @@
     </link>
     <gazebo reference="${fb}_${lr}_wheel">
+      <material>Gazebo/Black</material>
       <fdir1 value="1 0 0"/>
-      <material>Gazebo/Black</material>
       <mu1>1</mu1>
-      <mu2>0</mu2>
+      <mu2>1</mu2>
       <kp>1000000.0</kp>
-      <kd>1.0</kd>
-      <minDepth>0.01</minDepth>
-      <maxContacts>1</maxContacts>
+      <kd>10.0</kd>
+      <minDepth>0.001</minDepth>
       <turnGravityOff>false</turnGravityOff>
       <dampingFactor>0.01</dampingFactor>
