Commit message: Version 0.6.0
Added kinematics model
Fixed issue with launch files

File: catbot_description/urdf/fourWD_catbot.urdf.xacro (robot description, xacro)
@@ -21,10 +21,4 @@
                 izz="0.0000001" />
         </inertial>
-        <visual>
-            <origin xyz="0 0 0" rpy="0 0 0" />
-            <geometry>
-                <box size="0.001 0.001 0.001" />
-            </geometry>
-        </visual>
     </link>
     <gazebo reference="base_footprint">

File: catbot_description/urdf/include/wheel.urdf.xacro (robot description, xacro)
@@ -38,13 +38,13 @@
     </link>
     <gazebo reference="${fb}_${lr}_wheel">
-      <material>Gazebo/Black</material>
-      <fdir1 value="1 0 0"/>
-      <mu1>1</mu1>
-      <mu2>1</mu2>
-      <kp>1000000.0</kp>
-      <kd>10.0</kd>
-      <minDepth>0.001</minDepth>
-      <turnGravityOff>false</turnGravityOff>
-      <dampingFactor>0.01</dampingFactor>
+        <kp value="100000000.0"/>
+        <kd value="1"/>
+        <minDepth value="0.005"/>
+        <mu1 value="1"/> <!-- 2.0 -->
+        <mu2 value="1"/> <!-- 0.5 -->
+        <fdir1 value="1 0 0"/>
+        <material>Gazebo/Black</material>
+        <turnGravityOff>false</turnGravityOff>
+        <dampingFactor>0.01</dampingFactor>
     </gazebo>
     <joint name="${fb}_${lr}_wheel_joint" type="continuous">
@@ -64,4 +64,5 @@
         <hardwareInterface>EffortJointInterface</hardwareInterface>
         <mechanicalReduction>1</mechanicalReduction>
+        <motorTorqueConstant>1</motorTorqueConstant>
       </actuator>
     </transmission>
